File: mcu_conn.kicad_sch (KiCad schematic)
At the start: 12 parts, among them J10 Conn_01x04_Pin, J8 Conn_01x01_Pin, J9 Conn_01x05_Pin, Q6 IRLML6344

Commit message: Assign footprints and part fields, switch C11 to an electrolytic
Same 65 parts and 35 nets as before. No wiring changed.

Schematic edits by Luke:
- C11 is now a polarized capacitor symbol, plus side on VDD.
- D1 value reads D_proc.

Field edits by Claude:
- Footprints on C1 to C11, D1, R1 to R4 and SW1, which had none.
- Manufacturer, part number, DigiKey link, datasheet and description on
  the 53 parts in the BOM.
- Q1 to Q6 value FDV305N, to match their part number field.
- R5 value 53.6 and R10 value 66.5, the nearest values in stock.
- Stale 249 and 124 ohm part fields on R5, R6, R10, R12, R13 replaced.

J8, J9, R15 and R16 still have no footprint. J10 still has a logo
footprint.

Co-Authored-By: Claude Opus 5.5 (1M context) <noreply@anthropic.com>
Parts:
- Q6: value IRLML6344 -> FDV305N
Changed lines of the file:
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@@
 			)
 		)
-		(property "Value" "IRLML6344"
+		(property "Value" "FDV305N"
 			(at 125.73 66.0399 0)
 			(show_name no)
