File: mcu_conn.kicad_sch (KiCad schematic)
At the start: 42 parts, among them J11 MD_MCU_PU_EN, J9 MD_MCU_EN, Q6 FDV305N, U2 Teensy4.1, U3 INA190A5IDDFR, U4 INA190A5IDDFR

Commit message: Match resistor part fields to their footprints
23 resistors on the sub-sheets sit on 0603 footprints but still named
0805 parts. Their part number, manufacturer, DigiKey link, datasheet and
description fields now name stocked 0603 parts:

- R15, R42, R43 (100k): Yageo RC0603FR-07100KL
- R27, R28, R33, R36, R37 (1k): Yageo RC0603FR-071KL
- R17, R18 (10k): Yageo RC0603FR-0710KL
- R29 to R32 (100): Panasonic ERJ-3EKF1000V
- R41 (10): Panasonic ERJ-3EKF10R0V
- R22 to R26, R49, R50 (0): Vishay CRCW06030000Z0EAHP
- R34 (2.2): Panasonic ERJ-3RQF2R2V

R16, R35, R38 (9k) go back to the 0805 footprint, because no exact 9k
0603 part was found in stock. Their part stays Yageo RT0805BRE079KL.

No value or net changes.

Co-Authored-By: Claude Opus 5.5 (1M context) <noreply@anthropic.com>
Parts:
- R17, R18: Distributer Link 1 https://www.digikey.com/en/products/detail/yageo/RC0805FR-0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 -> https://www.digikey.com/en/products/detail/yageo/RC0603FR-0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; Manufacturer Part Number RC0805FR-0710KL -> RC0603FR-0710KL
- R22, R23, R24, R25, R26: Distributer Link 1 https://www.digikey.com/en/products/detail/vishay-dale/CRCW08050000Z0EAHP/2222316 -> https://www.digikey.com/en/products/detail/vishay-dale/CRCW06030000Z0EAHP/2222231; Manufacturer Part Number CRCW08050000Z0EAHP -> CRCW06030000Z0EAHP
- R27, R28: Distributer Link 1 https://www.digikey.com/en/products/detail/yageo/RC0805FR-0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 -> https://www.digikey.com/en/products/detail/yageo/RC0603FR-0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; Manufacturer Part Number RC0805FR-071KL -> RC0603FR-071KL
- R29, R30, R31, R32: Distributer Link 1 https://www.digikey.com/en/products/detail/yageo/RC0805FR-0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 -> https://www.digikey.com/en/products/detail/panasonic-indust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; Manufacturer YAGEO -> Panasonic Industry; Manufacturer Part Number RC0805FR-07100RL -> ERJ-3EKF1000V
Changed lines of the file:
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@@
 			)
 		)
-		(property "Description" "RES 1K OHM 1% 1/8W 0805"
+		(property "Description" "RES 1K OHM 1% 1/10W 0603"
 			(at 91.44 129.54 0)
 			(hide yes)
@@
 			)
 		)
-		(property "Manufacturer Part Number" "RC0805FR-071KL"
+		(property "Manufacturer Part Number" "RC0603FR-071KL"
 			(at 91.44 129.54 0)
 			(hide yes)
@@
 			)
 		)
-		(property "Distributer Link 1" "https://www.digikey.com/en/products/detail/yageo/RC0805FR-071KL/727444"
+		(property "Distributer Link 1" "https://www.digikey.com/en/products/detail/yageo/RC0603FR-071KL/726843"
 			(at 91.44 129.54 0)
 			(hide yes)
@@
 			)
 		)
-		(property "Description" "Resistor"
+		(property "Description" "RES 0 OHM JUMPER 1/3W 0603"
 			(at 204.47 99.06 0)
 			(hide yes)
@@
 			)
 		)
-		(property "Distributer Link 1" "https://www.digikey.com/en/products/detail/vishay-dale/CRCW08050000Z0EAHP/2222316"
+		(property "Distributer Link 1" "https://www.digikey.com/en/products/detail/vishay-dale/CRCW06030000Z0EAHP/2222231"
 			(at 204.47 99.06 0)
 			(hide yes)
@@
 			)
 		)
-		(property "Manufacturer Part Number" "CRCW08050000Z0EAHP"
+		(property "Manufacturer Part Number" "CRCW06030000Z0EAHP"
 			(at 204.47 99.06 0)
 			(hide yes)
@@
 			)
 		)
-		(property "Description" "Resistor"
+		(property "Description" "RES 0 OHM JUMPER 1/3W 0603"
 			(at 204.47 96.52 0)
 			(hide yes)
@@
 			)
 		)
-		(property "Distributer Link 1" "https://www.digikey.com/en/products/detail/vishay-dale/CRCW08050000Z0EAHP/2222316"
+		(property "Distributer Link 1" "https://www.digikey.com/en/products/detail/vishay-dale/CRCW06030000Z0EAHP/2222231"
 			(at 204.47 96.52 0)
 			(hide yes)
@@
 			)
 		)
-		(property "Manufacturer Part Number" "CRCW08050000Z0EAHP"
+		(property "Manufacturer Part Number" "CRCW06030000Z0EAHP"
 			(at 204.47 96.52 0)
 			(hide yes)
@@
 			)
 		)
-		(property "Datasheet" "https://yageogroup.com/content/datasheet/asset/file/PYU-RC_GROUP_51_ROHS_L"
+		(property "Datasheet" "https://industrial.panasonic.com/cdbs/www-data/pdf/RDA0000/AOA0000C304.pdf"
 			(at 41.91 140.97 0)
 			(hide yes)
@@
 			)
 		)
-		(property "Description" "RES 100 OHM 1% 1/8W 0805"
+		(property "Description" "RES 100 OHM 1% 1/10W 0603"
 			(at 41.91 140.97 0)
 			(hide yes)
@@
 			)
 		)
-		(property "Manufacturer" "YAGEO"
+		(property "Manufacturer" "Panasonic Industry"
 			(at 41.91 140.97 0)
 			(hide yes)
@@
 			)
 		)
-		(property "Manufacturer Part Number" "RC0805FR-07100RL"
+		(property "Manufacturer Part Number" "ERJ-3EKF1000V"
 			(at 41.91 140.97 0)
 			(hide yes)
@@
 			)
 		)
-		(property "Distributer Link 1" "https://www.digikey.com/en/products/detail/yageo/RC0805FR-07100RL/727543"
+		(property "Distributer Link 1" "https://www.digikey.com/en/products/detail/panasonic-industry/ERJ-3EKF1000V/196074"
 			(at 41.91 140.97 0)
 			(hide yes)
@@
 			)
 		)
-		(property "Description" "Resistor"
+		(property "Description" "RES 0 OHM JUMPER 1/3W 0603"
 			(at 204.47 106.68 0)
 			(hide yes)
@@
 			)
 		)
-		(property "Distributer Link 1" "https://www.digikey.com/en/products/detail/vishay-dale/CRCW08050000Z0EAHP/2222316"
+		(property "Distributer Link 1" "https://www.digikey.com/en/products/detail/vishay-dale/CRCW06030000Z0EAHP/2222231"
 			(at 204.47 106.68 0)
 			(hide yes)
@@
 			)
 		)
-		(property "Manufacturer Part Number" "CRCW08050000Z0EAHP"
+		(property "Manufacturer Part Number" "CRCW06030000Z0EAHP"
 			(at 204.47 106.68 0)
 			(hide yes)
@@
 			)
 		)
-		(property "Description" "Resistor"
+		(property "Description" "RES 0 OHM JUMPER 1/3W 0603"
 			(at 204.47 104.14 0)
 			(hide yes)
@@
 			)
 		)
-		(property "Distributer Link 1" "https://www.digikey.com/en/products/detail/vishay-dale/CRCW08050000Z0EAHP/2222316"
+		(property "Distributer Link 1" "https://www.digikey.com/en/products/detail/vishay-dale/CRCW06030000Z0EAHP/2222231"
 			(at 204.47 104.14 0)
 			(hide yes)
@@
 			)
 		)
-		(property "Manufacturer Part Number" "CRCW08050000Z0EAHP"
+		(property "Manufacturer Part Number" "CRCW06030000Z0EAHP"
 			(at 204.47 104.14 0)
 			(hide yes)
@@
 			)
 		)
-		(property "Datasheet" "https://yageogroup.com/content/datasheet/asset/file/PYU-RC_GROUP_51_ROHS_L"
+		(property "Datasheet" "https://industrial.panasonic.com/cdbs/www-data/pdf/RDA0000/AOA0000C304.pdf"
 			(at 41.91 163.83 0)
 			(hide yes)
@@
 			)
 		)
-		(property "Description" "RES 100 OHM 1% 1/8W 0805"
+		(property "Description" "RES 100 OHM 1% 1/10W 0603"
 			(at 41.91 163.83 0)
 			(hide yes)
@@
 			)
 		)
-		(property "Manufacturer" "YAGEO"
+		(property "Manufacturer" "Panasonic Industry"
 			(at 41.91 163.83 0)
 			(hide yes)
@@
 			)
 		)
-		(property "Manufacturer Part Number" "RC0805FR-07100RL"
+		(property "Manufacturer Part Number" "ERJ-3EKF1000V"
 			(at 41.91 163.83 0)
 			(hide yes)
@@
 			)
 		)
-		(property "Distributer Link 1" "https://www.digikey.com/en/products/detail/yageo/RC0805FR-07100RL/727543"
+		(property "Distributer Link 1" "https://www.digikey.com/en/products/detail/panasonic-industry/ERJ-3EKF1000V/196074"
 			(at 41.91 163.83 0)
 			(hide yes)
@@
 			)
 		)
-		(property "Description" "Resistor"
+		(property "Description" "RES 0 OHM JUMPER 1/3W 0603"
 			(at 204.47 101.6 0)
 			(hide yes)
@@
 			)
 		)
-		(property "Distributer Link 1" "https://www.digikey.com/en/products/detail/vishay-dale/CRCW08050000Z0EAHP/2222316"
+		(property "Distributer Link 1" "https://www.digikey.com/en/products/detail/vishay-dale/CRCW06030000Z0EAHP/2222231"
 			(at 204.47 101.6 0)
 			(hide yes)
@@
 			)
 		)
-		(property "Manufacturer Part Number" "CRCW08050000Z0EAHP"
+		(property "Manufacturer Part Number" "CRCW06030000Z0EAHP"
 			(at 204.47 101.6 0)
 			(hide yes)
@@
 			)
 		)
-		(property "Description" "RES 10K OHM 1% 1/8W 0805"
+		(property "Description" "RES 10K OHM 1% 1/10W 0603"
 			(at 168.91 71.12 0)
 			(hide yes)
@@
 			)
 		)
-		(property "Manufacturer Part Number" "RC0805FR-0710KL"
+		(property "Manufacturer Part Number" "RC0603FR-0710KL"
 			(at 168.91 71.12 0)
 			(hide yes)
@@
 			)
 		)
-		(property "Distributer Link 1" "https://www.digikey.com/en/products/detail/yageo/RC0805FR-0710KL/727535"
+		(property "Distributer Link 1" "https://www.digikey.com/en/products/detail/yageo/RC0603FR-0710KL/726880"
 			(at 168.91 71.12 0)
 			(hide yes)
@@
 			)
 		)
-		(property "Datasheet" "https://yageogroup.com/content/datasheet/asset/file/PYU-RC_GROUP_51_ROHS_L"
+		(property "Datasheet" "https://industrial.panasonic.com/cdbs/www-data/pdf/RDA0000/AOA0000C304.pdf"
 			(at 41.91 123.19 0)
 			(hide yes)
@@
 			)
 		)
-		(property "Description" "RES 100 OHM 1% 1/8W 0805"
+		(property "Description" "RES 100 OHM 1% 1/10W 0603"
 			(at 41.91 123.19 0)
 			(hide yes)
@@
 			)
 		)
-		(property "Manufacturer" "YAGEO"
+		(property "Manufacturer" "Panasonic Industry"
 			(at 41.91 123.19 0)
 			(hide yes)
@@
 			)
 		)
-		(property "Manufacturer Part Number" "RC0805FR-07100RL"
+		(property "Manufacturer Part Number" "ERJ-3EKF1000V"
 			(at 41.91 123.19 0)
 			(hide yes)
@@
 			)
 		)
-		(property "Distributer Link 1" "https://www.digikey.com/en/products/detail/yageo/RC0805FR-07100RL/727543"
+		(property "Distributer Link 1" "https://www.digikey.com/en/products/detail/panasonic-industry/ERJ-3EKF1000V/196074"
 			(at 41.91 123.19 0)
 			(hide yes)
@@
 			)
 		)
-		(property "Description" "RES 10K OHM 1% 1/8W 0805"
+		(property "Description" "RES 10K OHM 1% 1/10W 0603"
 			(at 181.61 50.8 0)
 			(hide yes)
@@
 			)
 		)
-		(property "Manufacturer Part Number" "RC0805FR-0710KL"
+		(property "Manufacturer Part Number" "RC0603FR-0710KL"
 			(at 181.61 50.8 0)
 			(hide yes)
@@
 			)
 		)
-		(property "Distributer Link 1" "https://www.digikey.com/en/products/detail/yageo/RC0805FR-0710KL/727535"
+		(property "Distributer Link 1" "https://www.digikey.com/en/products/detail/yageo/RC0603FR-0710KL/726880"
 			(at 181.61 50.8 0)
 			(hide yes)
@@
 			)
 		)
-		(property "Description" "RES 1K OHM 1% 1/8W 0805"
+		(property "Description" "RES 1K OHM 1% 1/10W 0603"
 			(at 91.44 171.45 0)
 			(hide yes)
@@
 			)
 		)
-		(property "Manufacturer Part Number" "RC0805FR-071KL"
+		(property "Manufacturer Part Number" "RC0603FR-071KL"
 			(at 91.44 171.45 0)
 			(hide yes)
@@
 			)
 		)
-		(property "Distributer Link 1" "https://www.digikey.com/en/products/detail/yageo/RC0805FR-071KL/727444"
+		(property "Distributer Link 1" "https://www.digikey.com/en/products/detail/yageo/RC0603FR-071KL/726843"
 			(at 91.44 171.45 0)
 			(hide yes)
@@
 			)
 		)
-		(property "Datasheet" "https://yageogroup.com/content/datasheet/asset/file/PYU-RC_GROUP_51_ROHS_L"
+		(property "Datasheet" "https://industrial.panasonic.com/cdbs/www-data/pdf/RDA0000/AOA0000C304.pdf"
 			(at 41.91 184.15 0)
 			(hide yes)
@@
 			)
 		)
-		(property "Description" "RES 100 OHM 1% 1/8W 0805"
+		(property "Description" "RES 100 OHM 1% 1/10W 0603"
 			(at 41.91 184.15 0)
 			(hide yes)
@@
 			)
 		)
-		(property "Manufacturer" "YAGEO"
+		(property "Manufacturer" "Panasonic Industry"
 			(at 41.91 184.15 0)
 			(hide yes)
@@
 			)
 		)
-		(property "Manufacturer Part Number" "RC0805FR-07100RL"
+		(property "Manufacturer Part Number" "ERJ-3EKF1000V"
 			(at 41.91 184.15 0)
 			(hide yes)
@@
 			)
 		)
-		(property "Distributer Link 1" "https://www.digikey.com/en/products/detail/yageo/RC0805FR-07100RL/727543"
+		(property "Distributer Link 1" "https://www.digikey.com/en/products/detail/panasonic-industry/ERJ-3EKF1000V/196074"
 			(at 41.91 184.15 0)
 			(hide yes)
