File: tmp_sense.kicad_sch (KiCad schematic)
At the start: 0 parts

Commit message: Add the title block to the MCU and temperature sheets
Both sub-sheets now carry the same title, date, revision and four author
names as the top sheet. No parts or nets change.
Other:
- title: (none) -> EE372 LDO bringup board
Changed lines of the file:
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@@
 	(generator_version "10.0")
 	(paper "A4")
+	(title_block
+		(title "EE372 LDO bringup board")
+		(date "2026-08-02")
+		(rev "0")
+		(comment 1 "Luke Qiao")
+		(comment 2 "Spencer Wallace")
+		(comment 3 "Luis Sanchez")
+		(comment 4 "Caleb Ketchum")
+	)
 	(bus
 		(pts
