File: noise_amp.kicad_sch (KiCad schematic)
At the start: 25 parts, among them J16 NOISE_X100, J17 NOISE_X1000, U5 OPA4388IDR

Commit message: Point R16, R35, R38 at a stocked 9k part
Part number, DigiKey link, datasheet and description fields now name
Yageo RT0805BRE079KL (9k, 0.1%, thin film, 0805). The fields still named
the 10k part after the value change. No value, footprint or net changes.

Co-Authored-By: Claude Opus 5.5 (1M context) <noreply@anthropic.com>
Parts:
- R16, R35, R38: Distributer Link 1 https://www.digikey.com/en/products/detail/yageo/RC0805FR-0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 -> https://www.digikey.com/en/products/detail/yageo/RT0805BRE0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; Manufacturer Part Number RC0805FR-0710KL -> RT0805BRE079KL
Changed lines of the file:
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@@
 			)
 		)
-		(property "Datasheet" "https://yageogroup.com/content/datasheet/asset/file/PYU-RC_GROUP_51_ROHS_L"
+		(property "Datasheet" "https://yageogroup.com/content/datasheet/asset/file/PYU-RT_1-TO-0-01_ROHS_L"
 			(at 153.67 71.12 0)
 			(hide yes)
@@
 			)
 		)
-		(property "Description" "RES 10K OHM 1% 1/8W 0805"
+		(property "Description" "RES 9K OHM 0.1% 1/8W 0805 THIN FILM"
 			(at 153.67 71.12 0)
 			(hide yes)
@@
 			)
 		)
-		(property "Distributer Link 1" "https://www.digikey.com/en/products/detail/yageo/RC0805FR-0710KL/727535"
+		(property "Distributer Link 1" "https://www.digikey.com/en/products/detail/yageo/RT0805BRE079KL/5932404"
 			(at 153.67 71.12 0)
 			(hide yes)
@@
 			)
 		)
-		(property "Manufacturer Part Number" "RC0805FR-0710KL"
+		(property "Manufacturer Part Number" "RT0805BRE079KL"
 			(at 153.67 71.12 0)
 			(hide yes)
@@
 			)
 		)
-		(property "Datasheet" "https://yageogroup.com/content/datasheet/asset/file/PYU-RC_GROUP_51_ROHS_L"
+		(property "Datasheet" "https://yageogroup.com/content/datasheet/asset/file/PYU-RT_1-TO-0-01_ROHS_L"
 			(at 154.94 124.46 0)
 			(hide yes)
@@
 			)
 		)
-		(property "Description" "RES 10K OHM 1% 1/8W 0805"
+		(property "Description" "RES 9K OHM 0.1% 1/8W 0805 THIN FILM"
 			(at 154.94 124.46 0)
 			(hide yes)
@@
 			)
 		)
-		(property "Distributer Link 1" "https://www.digikey.com/en/products/detail/yageo/RC0805FR-0710KL/727535"
+		(property "Distributer Link 1" "https://www.digikey.com/en/products/detail/yageo/RT0805BRE079KL/5932404"
 			(at 154.94 124.46 0)
 			(hide yes)
@@
 			)
 		)
-		(property "Manufacturer Part Number" "RC0805FR-0710KL"
+		(property "Manufacturer Part Number" "RT0805BRE079KL"
 			(at 154.94 124.46 0)
 			(hide yes)
@@
 			)
 		)
-		(property "Datasheet" "https://yageogroup.com/content/datasheet/asset/file/PYU-RC_GROUP_51_ROHS_L"
+		(property "Datasheet" "https://yageogroup.com/content/datasheet/asset/file/PYU-RT_1-TO-0-01_ROHS_L"
 			(at 124.46 71.12 0)
 			(hide yes)
@@
 			)
 		)
-		(property "Description" "RES 10K OHM 1% 1/8W 0805"
+		(property "Description" "RES 9K OHM 0.1% 1/8W 0805 THIN FILM"
 			(at 124.46 71.12 0)
 			(hide yes)
@@
 			)
 		)
-		(property "Distributer Link 1" "https://www.digikey.com/en/products/detail/yageo/RC0805FR-0710KL/727535"
+		(property "Distributer Link 1" "https://www.digikey.com/en/products/detail/yageo/RT0805BRE079KL/5932404"
 			(at 124.46 71.12 0)
 			(hide yes)
@@
 			)
 		)
-		(property "Manufacturer Part Number" "RC0805FR-0710KL"
+		(property "Manufacturer Part Number" "RT0805BRE079KL"
 			(at 124.46 71.12 0)
 			(hide yes)
