File: noise_amp.kicad_sch (KiCad schematic)
At the start: 25 parts, among them J16 NOISE_X100, J17 NOISE_X1000, U5 OPA4388IDR

Commit message: Match resistor part fields to their footprints
23 resistors on the sub-sheets sit on 0603 footprints but still named
0805 parts. Their part number, manufacturer, DigiKey link, datasheet and
description fields now name stocked 0603 parts:

- R15, R42, R43 (100k): Yageo RC0603FR-07100KL
- R27, R28, R33, R36, R37 (1k): Yageo RC0603FR-071KL
- R17, R18 (10k): Yageo RC0603FR-0710KL
- R29 to R32 (100): Panasonic ERJ-3EKF1000V
- R41 (10): Panasonic ERJ-3EKF10R0V
- R22 to R26, R49, R50 (0): Vishay CRCW06030000Z0EAHP
- R34 (2.2): Panasonic ERJ-3RQF2R2V

R16, R35, R38 (9k) go back to the 0805 footprint, because no exact 9k
0603 part was found in stock. Their part stays Yageo RT0805BRE079KL.

No value or net changes.

Co-Authored-By: Claude Opus 5.5 (1M context) <noreply@anthropic.com>
Parts:
- R15, R42, R43: Distributer Link 1 https://www.digikey.com/en/products/detail/yageo/RC0805FR-0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 -> https://www.digikey.com/en/products/detail/yageo/RC0603FR-0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; Manufacturer Part Number RC0805FR-07100KL -> RC0603FR-07100KL
- R16, R35, R38: footprint Resistor_SMD:R_0603_1608Metric_Pad0.98x0.95mm_HandSolder -> Resistor_SMD:R_0805_2012Metric_Pad1.20x1.40mm_HandSolder
- R33, R36, R37: Distributer Link 1 https://www.digikey.com/en/products/detail/yageo/RC0805FR-0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 -> https://www.digikey.com/en/products/detail/yageo/RC0603FR-0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; Manufacturer Part Number RC0805FR-071KL -> RC0603FR-071KL
- R41: Distributer Link 1 https://www.digikey.com/en/products/result?keywords=RC0805F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 -> https://www.digikey.com/en/products/detail/panasonic-indust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; Manufacturer YAGEO -> Panasonic Industry; Manufacturer Part Number RC0805FR-0710RL -> ERJ-3EKF10R0V
- R49, R50: Distributer Link 1 https://www.digikey.com/en/products/detail/vishay-dale/CRCW08050000Z0EAHP/2222316 -> https://www.digikey.com/en/products/detail/vishay-dale/CRCW06030000Z0EAHP/2222231; Manufacturer Part Number CRCW08050000Z0EAHP -> CRCW06030000Z0EAHP
Changed lines of the file:
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@@
 			)
 		)
-		(property "Datasheet" "https://yageogroup.com/content/datasheet/asset/file/PYU-RC_GROUP_51_ROHS_L"
+		(property "Datasheet" "https://industrial.panasonic.com/cdbs/www-data/pdf/RDA0000/AOA0000C304.pdf"
 			(at 29.21 59.69 0)
 			(hide yes)
@@
 			)
 		)
-		(property "Description" "RES 10 OHM 1% 1/8W 0805"
+		(property "Description" "RES 10 OHM 1% 1/10W 0603"
 			(at 29.21 59.69 0)
 			(hide yes)
@@
 			)
 		)
-		(property "Distributer Link 1" "https://www.digikey.com/en/products/result?keywords=RC0805FR-0710RL"
+		(property "Distributer Link 1" "https://www.digikey.com/en/products/detail/panasonic-industry/ERJ-3EKF10R0V/603878"
 			(at 29.21 59.69 0)
 			(hide yes)
@@
 			)
 		)
-		(property "Manufacturer Part Number" "RC0805FR-0710RL"
+		(property "Manufacturer Part Number" "ERJ-3EKF10R0V"
 			(at 29.21 59.69 0)
 			(hide yes)
@@
 			)
 		)
-		(property "Manufacturer" "YAGEO"
+		(property "Manufacturer" "Panasonic Industry"
 			(at 29.21 59.69 0)
 			(hide yes)
@@
 			)
 		)
-		(property "Description" "RES 1K OHM 1% 1/8W 0805"
+		(property "Description" "RES 1K OHM 1% 1/10W 0603"
 			(at 114.3 77.47 0)
 			(hide yes)
@@
 			)
 		)
-		(property "Distributer Link 1" "https://www.digikey.com/en/products/detail/yageo/RC0805FR-071KL/727444"
+		(property "Distributer Link 1" "https://www.digikey.com/en/products/detail/yageo/RC0603FR-071KL/726843"
 			(at 114.3 77.47 0)
 			(hide yes)
@@
 			)
 		)
-		(property "Manufacturer Part Number" "RC0805FR-071KL"
+		(property "Manufacturer Part Number" "RC0603FR-071KL"
 			(at 114.3 77.47 0)
 			(hide yes)
@@
 			)
 		)
-		(property "Footprint" "Resistor_SMD:R_0603_1608Metric_Pad0.98x0.95mm_HandSolder"
+		(property "Footprint" "Resistor_SMD:R_0805_2012Metric_Pad1.20x1.40mm_HandSolder"
 			(at 153.67 72.898 90)
 			(hide yes)
@@
 			)
 		)
-		(property "Description" "RES 100K OHM 1% 1/8W 0805"
+		(property "Description" "RES 100K OHM 1% 1/10W 0603"
 			(at 69.85 83.82 0)
 			(hide yes)
@@
 			)
 		)
-		(property "Distributer Link 1" "https://www.digikey.com/en/products/detail/yageo/RC0805FR-07100KL/1960237"
+		(property "Distributer Link 1" "https://www.digikey.com/en/products/detail/yageo/RC0603FR-07100KL/726889"
 			(at 69.85 83.82 0)
 			(hide yes)
@@
 			)
 		)
-		(property "Manufacturer Part Number" "RC0805FR-07100KL"
+		(property "Manufacturer Part Number" "RC0603FR-07100KL"
 			(at 69.85 83.82 0)
 			(hide yes)
@@
 			)
 		)
-		(property "Description" "RES 1K OHM 1% 1/8W 0805"
+		(property "Description" "RES 1K OHM 1% 1/10W 0603"
 			(at 142.24 130.81 0)
 			(hide yes)
@@
 			)
 		)
-		(property "Distributer Link 1" "https://www.digikey.com/en/products/detail/yageo/RC0805FR-071KL/727444"
+		(property "Distributer Link 1" "https://www.digikey.com/en/products/detail/yageo/RC0603FR-071KL/726843"
 			(at 142.24 130.81 0)
 			(hide yes)
@@
 			)
 		)
-		(property "Manufacturer Part Number" "RC0805FR-071KL"
+		(property "Manufacturer Part Number" "RC0603FR-071KL"
 			(at 142.24 130.81 0)
 			(hide yes)
@@
 			)
 		)
-		(property "Description" "Resistor"
+		(property "Description" "RES 0 OHM JUMPER 1/3W 0603"
 			(at 168.91 113.03 0)
 			(hide yes)
@@
 			)
 		)
-		(property "Distributer Link 1" "https://www.digikey.com/en/products/detail/vishay-dale/CRCW08050000Z0EAHP/2222316"
+		(property "Distributer Link 1" "https://www.digikey.com/en/products/detail/vishay-dale/CRCW06030000Z0EAHP/2222231"
 			(at 168.91 113.03 0)
 			(hide yes)
@@
 			)
 		)
-		(property "Manufacturer Part Number" "CRCW08050000Z0EAHP"
+		(property "Manufacturer Part Number" "CRCW06030000Z0EAHP"
 			(at 168.91 113.03 0)
 			(hide yes)
@@
 			)
 		)
-		(property "Footprint" "Resistor_SMD:R_0603_1608Metric_Pad0.98x0.95mm_HandSolder"
+		(property "Footprint" "Resistor_SMD:R_0805_2012Metric_Pad1.20x1.40mm_HandSolder"
 			(at 154.94 126.238 90)
 			(hide yes)
@@
 			)
 		)
-		(property "Description" "Resistor"
+		(property "Description" "RES 0 OHM JUMPER 1/3W 0603"
 			(at 168.91 59.69 0)
 			(hide yes)
@@
 			)
 		)
-		(property "Distributer Link 1" "https://www.digikey.com/en/products/detail/vishay-dale/CRCW08050000Z0EAHP/2222316"
+		(property "Distributer Link 1" "https://www.digikey.com/en/products/detail/vishay-dale/CRCW06030000Z0EAHP/2222231"
 			(at 168.91 59.69 0)
 			(hide yes)
@@
 			)
 		)
-		(property "Manufacturer Part Number" "CRCW08050000Z0EAHP"
+		(property "Manufacturer Part Number" "CRCW06030000Z0EAHP"
 			(at 168.91 59.69 0)
 			(hide yes)
@@
 			)
 		)
-		(property "Description" "RES 1K OHM 1% 1/8W 0805"
+		(property "Description" "RES 1K OHM 1% 1/10W 0603"
 			(at 140.97 77.47 0)
 			(hide yes)
@@
 			)
 		)
-		(property "Distributer Link 1" "https://www.digikey.com/en/products/detail/yageo/RC0805FR-071KL/727444"
+		(property "Distributer Link 1" "https://www.digikey.com/en/products/detail/yageo/RC0603FR-071KL/726843"
 			(at 140.97 77.47 0)
 			(hide yes)
@@
 			)
 		)
-		(property "Manufacturer Part Number" "RC0805FR-071KL"
+		(property "Manufacturer Part Number" "RC0603FR-071KL"
 			(at 140.97 77.47 0)
 			(hide yes)
@@
 			)
 		)
-		(property "Footprint" "Resistor_SMD:R_0603_1608Metric_Pad0.98x0.95mm_HandSolder"
+		(property "Footprint" "Resistor_SMD:R_0805_2012Metric_Pad1.20x1.40mm_HandSolder"
 			(at 124.46 72.898 90)
 			(hide yes)
@@
 			)
 		)
-		(property "Description" "RES 100K OHM 1% 1/8W 0805"
+		(property "Description" "RES 100K OHM 1% 1/10W 0603"
 			(at 104.14 64.77 0)
 			(hide yes)
@@
 			)
 		)
-		(property "Distributer Link 1" "https://www.digikey.com/en/products/detail/yageo/RC0805FR-07100KL/1960237"
+		(property "Distributer Link 1" "https://www.digikey.com/en/products/detail/yageo/RC0603FR-07100KL/726889"
 			(at 104.14 64.77 0)
 			(hide yes)
@@
 			)
 		)
-		(property "Manufacturer Part Number" "RC0805FR-07100KL"
+		(property "Manufacturer Part Number" "RC0603FR-07100KL"
 			(at 104.14 64.77 0)
 			(hide yes)
@@
 			)
 		)
-		(property "Description" "RES 100K OHM 1% 1/8W 0805"
+		(property "Description" "RES 100K OHM 1% 1/10W 0603"
 			(at 69.85 71.12 0)
 			(hide yes)
@@
 			)
 		)
-		(property "Distributer Link 1" "https://www.digikey.com/en/products/detail/yageo/RC0805FR-07100KL/1960237"
+		(property "Distributer Link 1" "https://www.digikey.com/en/products/detail/yageo/RC0603FR-07100KL/726889"
 			(at 69.85 71.12 0)
 			(hide yes)
@@
 			)
 		)
-		(property "Manufacturer Part Number" "RC0805FR-07100KL"
+		(property "Manufacturer Part Number" "RC0603FR-07100KL"
 			(at 69.85 71.12 0)
 			(hide yes)
