File: noise_amp.kicad_sch (KiCad schematic)
At the start: 25 parts, among them J16 NOISE_X100, J17 NOISE_X1000, U5 OPA4388IDR

Commit message: Add bring-up notes to the schematic
Text notes only, no parts or nets change. Leave R3, R21, R29 to R32,
R40, R44 and R55 off at first. Possibly lift C6 and C11 when driving
VIN from the buffer. Add a large pull-down on the buffer input.
Other:
- note added: "Initially leave off R44"
Changed lines of the file:
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@@
+		)
+	)
+	(text "Initially leave off R44"
+		(exclude_from_sim yes)
+		(at 44.45 41.148 0)
+		(effects
+			(font
+				(size 1.27 1.27)
+			)
+			(justify left)
 		)
 	)
