File: buffer.kicad_sch (KiCad schematic)
At the start: 5 parts, among them J12 BUF_EN, U6 BUF602ID

Commit message: Standardized resistor footprints
Parts:
- R34: footprint Resistor_SMD:R_0805_2012Metric_Pad1.20x1.40mm_HandSolder -> Resistor_SMD:R_0603_1608Metric_Pad0.98x0.95mm_HandSolder
Changed lines of the file:
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@@
 			)
 		)
-		(property "Footprint" "Resistor_SMD:R_0805_2012Metric_Pad1.20x1.40mm_HandSolder"
+		(property "Footprint" "Resistor_SMD:R_0603_1608Metric_Pad0.98x0.95mm_HandSolder"
 			(at 60.96 80.518 90)
 			(hide yes)
