File: buffer.kicad_sch (KiCad schematic)
At the start: 5 parts, among them J12 BUF_EN, U6 BUF602ID

Commit message: Match resistor part fields to their footprints
23 resistors on the sub-sheets sit on 0603 footprints but still named
0805 parts. Their part number, manufacturer, DigiKey link, datasheet and
description fields now name stocked 0603 parts:

- R15, R42, R43 (100k): Yageo RC0603FR-07100KL
- R27, R28, R33, R36, R37 (1k): Yageo RC0603FR-071KL
- R17, R18 (10k): Yageo RC0603FR-0710KL
- R29 to R32 (100): Panasonic ERJ-3EKF1000V
- R41 (10): Panasonic ERJ-3EKF10R0V
- R22 to R26, R49, R50 (0): Vishay CRCW06030000Z0EAHP
- R34 (2.2): Panasonic ERJ-3RQF2R2V

R16, R35, R38 (9k) go back to the 0805 footprint, because no exact 9k
0603 part was found in stock. Their part stays Yageo RT0805BRE079KL.

No value or net changes.

Co-Authored-By: Claude Opus 5.5 (1M context) <noreply@anthropic.com>
Parts:
- R34: Distributer Link 1 https://www.digikey.com/en/products/result?keywords=ERJ-6RQ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 -> https://www.digikey.com/en/products/detail/panasonic-indust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; Manufacturer Part Number ERJ-6RQF2R2V -> ERJ-3RQF2R2V
Changed lines of the file:
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@@
 			)
 		)
-		(property "Description" "RES 2.2 OHM 1% 1/8W 0805"
+		(property "Description" "RES 2.2 OHM 1% 1/10W 0603"
 			(at 60.96 78.74 0)
 			(hide yes)
@@
 			)
 		)
-		(property "Manufacturer Part Number" "ERJ-6RQF2R2V"
+		(property "Manufacturer Part Number" "ERJ-3RQF2R2V"
 			(at 60.96 78.74 0)
 			(hide yes)
@@
 			)
 		)
-		(property "Distributer Link 1" "https://www.digikey.com/en/products/result?keywords=ERJ-6RQF2R2V"
+		(property "Distributer Link 1" "https://www.digikey.com/en/products/detail/panasonic-industry/ERJ-3RQF2R2V/308066"
 			(at 60.96 78.74 0)
 			(hide yes)
