File: ldo_bringup_board_ee372.kicad_pcb (KiCad board)
At the start: 4 copper layers, 100 x 100 mm, 152 parts, among them J1 VIN, J10 MD_SW_EN, J11 MD_MCU_PU_EN, J12 BUF_EN, J13 VSIG, J14 VSIG_BUF, J15 NR, J16 NOISE_X100, J17 NOISE_X1000, J18 VIN_PROBE, J19 VREF_PROBE, J2 GND, J20 VOUT_PROBE, J21 VG0_PROBE, J22 VG1_PROBE, J23 VG2_PROBE, J24 VG3_PROBE, J25 VG4_PROBE, J3 IBIAS, J4 VOUT, J5 VIN_SMA, J6 VOUT_SMA, J7 GND, J8 5V, J9 MD_MCU_EN, Q1 FDV305N, Q2 FDV305N, Q3 FDV305N, Q4 FDV305N, Q5 FDV305N, Q6 FDV305N, SW1 MD_SW, U1 LDO_DualMode_BGR_EE372, U2 Teensy4.1, U3 INA190A5IDDFR, U4 INA190A5IDDFR, U5 OPA4388IDR, U6 BUF602ID, U7 ADT7310TRZ

Commit message: Add seven ground test points, TP22 to TP25 and TP31 to TP33
Keystone 5006 on GND in the schematic, footprints added to the PCB and
parked outside the board outline. Not placed yet, so DRC shows them
unconnected.
Parts:
- added TP22: GND, TestPoint:TestPoint_Keystone_5005-5009_Compact, F.Cu at (225.5, 70.5)
- added TP23: GND, TestPoint:TestPoint_Keystone_5005-5009_Compact, F.Cu at (225.5, 75.6)
- added TP24: GND, TestPoint:TestPoint_Keystone_5005-5009_Compact, F.Cu at (225.5, 80.6)
- added TP25: GND, TestPoint:TestPoint_Keystone_5005-5009_Compact, F.Cu at (225.5, 85.7)
- added TP31: GND, TestPoint:TestPoint_Keystone_5005-5009_Compact, F.Cu at (230.6, 70.5)
- added TP32: GND, TestPoint:TestPoint_Keystone_5005-5009_Compact, F.Cu at (230.6, 75.6)
- added TP33: GND, TestPoint:TestPoint_Keystone_5005-5009_Compact, F.Cu at (230.6, 80.6)
