File: ldo_bringup_board_ee372.kicad_pcb (KiCad board)
At the start: 4 copper layers, 100 x 100 mm, 159 parts, among them J1 VIN, J10 MD_SW_EN, J11 MD_MCU_PU_EN, J12 BUF_EN, J13 VSIG, J14 VSIG_BUF, J15 NR, J16 NOISE_X100, J17 NOISE_X1000, J18 VIN_PROBE, J19 VREF_PROBE, J2 GND, J20 VOUT_PROBE, J21 VG0_PROBE, J22 VG1_PROBE, J23 VG2_PROBE, J24 VG3_PROBE, J25 VG4_PROBE, J3 IBIAS, J4 VOUT, J5 VIN_SMA, J6 VOUT_SMA, J7 GND, J8 5V, J9 MD_MCU_EN, Q1 FDV305N, Q2 FDV305N, Q3 FDV305N, Q4 FDV305N, Q5 FDV305N, Q6 FDV305N, SW1 MD_SW, U1 LDO_DualMode_BGR_EE372, U2 Teensy4.1, U3 INA190A5IDDFR, U4 INA190A5IDDFR, U5 OPA4388IDR, U6 BUF602ID, U7 ADT7310TRZ

Commit message: Place six of the new ground test points beside their signal test points
TP23 by TP1, TP24 by TP27, TP33 by TP14, TP22 by TP3, TP25 by TP28 and
TP31 by TP2, each 4.25 to 4.93 mm away. Four GND stitching vias that sat
under the new pads removed. Zones refilled. TP32 left parked.

Tracks unchanged. DRC 0 errors, schematic parity 0.

Co-Authored-By: Claude Opus 5.5 (1M context) <noreply@anthropic.com>
Parts:
- moved TP33 114.4 mm to (116.2, 77.0)
- moved TP22 96.5 mm to (129.2, 77.2)
- moved TP25 96.3 mm to (131.5, 106.5)
- moved TP31 91.5 mm to (143.0, 97.0)
- moved TP24 85.7 mm to (150.5, 122.0)
- moved TP23 84.4 mm to (141.2, 71.5)
Routing:
- net GND: vias 390 -> 386
Changed lines of the file:
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@@
 	(footprint "TestPoint:TestPoint_Keystone_5005-5009_Compact"
 		(layer "F.Cu")
-		(at 225.525 85.675)
+		(at 131.5 106.5)
 		(descr "Keystone THM Compact Test Point 5005-5009, http://www.keyelco.com/product-pdf.cfm?p=1314")
 		(tags "Through Hole Mount Test Points")
@@
 	(footprint "TestPoint:TestPoint_Keystone_5005-5009_Compact"
 		(layer "F.Cu")
-		(at 230.575 80.625)
+		(at 116.25 77)
 		(descr "Keystone THM Compact Test Point 5005-5009, http://www.keyelco.com/product-pdf.cfm?p=1314")
 		(tags "Through Hole Mount Test Points")
@@
 	(footprint "TestPoint:TestPoint_Keystone_5005-5009_Compact"
 		(layer "F.Cu")
-		(at 225.525 75.575)
+		(at 141.25 71.5)
 		(descr "Keystone THM Compact Test Point 5005-5009, http://www.keyelco.com/product-pdf.cfm?p=1314")
 		(tags "Through Hole Mount Test Points")
@@
 	(footprint "TestPoint:TestPoint_Keystone_5005-5009_Compact"
 		(layer "F.Cu")
-		(at 225.525 70.525)
+		(at 129.25 77.25)
 		(descr "Keystone THM Compact Test Point 5005-5009, http://www.keyelco.com/product-pdf.cfm?p=1314")
 		(tags "Through Hole Mount Test Points")
@@
 	(footprint "TestPoint:TestPoint_Keystone_5005-5009_Compact"
 		(layer "F.Cu")
-		(at 225.525 80.625)
+		(at 150.5 122)
 		(descr "Keystone THM Compact Test Point 5005-5009, http://www.keyelco.com/product-pdf.cfm?p=1314")
 		(tags "Through Hole Mount Test Points")
@@
 	(footprint "TestPoint:TestPoint_Keystone_5005-5009_Compact"
 		(layer "F.Cu")
-		(at 230.575 70.525)
+		(at 143 97)
 		(descr "Keystone THM Compact Test Point 5005-5009, http://www.keyelco.com/product-pdf.cfm?p=1314")
 		(tags "Through Hole Mount Test Points")
@@
 	)
 	(via
-		(at 117.4 77.9)
-		(size 0.6)
-		(drill 0.3)
-		(layers "F.Cu" "B.Cu")
-		(net "GND")
-	)
-	(via
 		(at 148.65 122.9)
 		(size 0.6)
@@
 	)
 	(via
-		(at 142.4 97.9)
-		(size 0.6)
-		(drill 0.3)
-		(layers "F.Cu" "B.Cu")
-		(net "GND")
-	)
-	(via
 		(at 192.4 72.9)
 		(size 0.6)
@@
 	)
 	(via
-		(at 142.4 72.9)
-		(size 0.6)
-		(drill 0.3)
-		(layers "F.Cu" "B.Cu")
-		(net "GND")
-	)
-	(via
 		(at 114.9 100.4)
 		(size 0.6)
@@
 		(size 0.6)
 		(drill 0.3)
-		(layers "F.Cu" "B.Cu")
-		(net "GND")
-	)
-	(via
-		(at 132.4 107.9)
-		(size 0.6)
-		(drill 0.3)
